File: video-thingy.kicad_pcb (KiCad board)
At the start: 4 copper layers, 88.9 x 97 mm, 56 parts, among them J1 RCJ-041, J2 RCJ-041, J3 RCJ-041, J4 RCJ-041, J5 RCJ-041, J6 RCJ-041, J7 RCJ-041, J8 RCJ-041, SW1 RotaryEncoder, SW10 Push_Button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

Commit message: Update pcb, for prod
Parts:
- added MOUNT: TestPoint_Pad_D1.0mm, TestPoint:TestPoint_Pad_D1.0mm, B.Cu at (201.6, 137.2)
- added MOUNT3: TestPoint_Pad_D1.0mm, TestPoint:TestPoint_Pad_D1.0mm, B.Cu at (200.6, 139.6)
- moved TP15 1.80 mm to (182.8, 132.8)
Routing:
- net GND: track 29.6 -> 56.9 mm, vias 20 -> 32
- net +5V: track 50.2 -> 55.3 mm, vias 13 -> 15
- net Net-(U8-GP2): track 6.46 -> 7.20 mm

Commit message: Routing optimization
Parts:
- removed the MOUNT at (201.6, 137.2)
- removed MOUNT3: TestPoint_Pad_D1.0mm, TestPoint:TestPoint_Pad_D1.0mm
Connections:
- D1 pad 3: +5V -> GND
- D2 pad 3: +5V -> GND
- D3 pad 3: +5V -> GND
- D4 pad 3: +5V -> GND
- D5 pad 3: +5V -> GND
- N1 pad 4: +5V -> GND
- R1 pad 1: +5V -> GND
- R22 pad 1: Net-(U2-X5) -> GND
- SW1 pad A: A1 -> GND
- SW10 pad 2: +5V -> GND
- SW11 pad 2: +5V -> GND
- SW12 pad 1: Net-(U8-GP12) -> GND
- SW12 pad 2: +5V -> GND
- SW13 pad 2: +5V -> GND
- U10 pad 4: +5V -> GND
- U10 pad 5: +5V -> GND
- U2 pad 16: +5V -> GND
- U2 pad 5: Net-(U2-X5) -> GND
- U3 pad 8: +5V -> GND
- U4 pad 8: +5V -> GND
- U5 pad 8: +5V -> GND
- U6 pad 16: GP7-A -> GND
- U7 pad 20: GP7-A -> GND
- U8 pad 10: A1 -> GND
- U8 pad 13: Net-(U8-GP12) -> GND
- U8 pad 23: +5V -> GND
- U9 pad 4: +5V -> GND
- U9 pad 5: +5V -> GND
Routing:
- net GND: track 56.9 -> 225.3 mm, vias 32 -> 30
- net A1: track 86.2 -> 0.00 mm, vias 1 -> 0
- net Net-(U8-GP12): track 60.7 -> 0.00 mm, vias 4 -> 0
- net +5V: track 55.3 -> 0.00 mm, vias 15 -> 0
- net GP7-A: track 39.1 -> 0.00 mm, vias 5 -> 0
- net Net-(U2-X5): track 24.2 -> 0.00 mm, vias 1 -> 0
- net +3.3V: track 147.3 -> 142.0 mm
- net Net-(U8-GP13): track 61.2 -> 57.0 mm
- net Net-(U8-GP10): track 67.6 -> 64.2 mm
- net PostProcessingMixed: track 130.7 -> 133.3 mm
- net B: track 42.8 -> 41.0 mm
- net Net-(C2-Pad2): track 53.8 -> 52.3 mm
- net AnalogL: track 117.5 -> 119.1 mm
- net RSET: track 19.6 -> 21.1 mm
- net A2: track 90.7 -> 92.2 mm
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
Commit message: Routing opti
Routing:
- net GND: track 225.3 -> 226.3 mm
